File: BenchBudEE/Power.sch (KiCad schematic (older format))
At the start: 0 parts

Commit message: Module 3 Unit 6
Understanding The Power Protection And Filtering Module
Parts:
- added C? (x2): C, ~, symbol C
- added F? (x4): FUSE, ~, symbol FUSE
- added L? (x2): INDUCTOR, ~, symbol INDUCTOR
- added P?: CONN_12X2, symbol CONN_12X2
- added R?: R, ~, symbol R
- added SW?: SWITCH_INV, ~, symbol SWITCH_INV
Connections:
- new net: F?.1, P?.10 (P10)
- new net: F?.1, P?.14 (P14)
- new net: P?.16 (P16), SW?.2
- new net: F?.1, P?.2 (P2)
- new net: F?.1, P?.4 (P4), P?.6 (P6)
- new net: R?.1, SW?.1
- new net +12P: F?.2, L?.1
- new net +12V: C?.1, L?.2
- new net +3.3V: F?.2, R?.2
- new net +5V: F?.2
- new net -12P: F?.2, L?.1
- new net -12V: C?.2, L?.2
- new net GND: C?.1, C?.2, P?.3 (P3), P?.5 (P5), SW?.3
